Commit message: tel updata

File: teleop_control/vendor/tianji/Marvin M6-S-L-CCS-696-V4.0 urdf (FUSION)/urdf/marvin_left_with_gripper.urdf (robot description, URDF)
Before this commit: robot marvin_l_with_gripper, 14 links, 13 joints
Joints:
- joint gripper_mount_L: origin xyz=0 0 0 rpy=0 0 0.785398163397 -> xyz=0 0 0 rpy=0 0 2.356194490192345

File: teleop_control/vendor/tianji/Marvin M6-S-R-CCS-696-V4.0 urdf (FUSION)/urdf/marvin_right_with_gripper.urdf (robot description, URDF)
Before this commit: robot marvin_r_with_gripper, 14 links, 13 joints
Joints:
- joint gripper_mount_R: origin xyz=0 0 0 rpy=0 0 0.785398163397 -> xyz=0 0 0 rpy=0 0 -0.7853981633974483

Commit message: Set gripper TCP, add simulation viewer, and share teleop heading

File: teleop_control/vendor/tianji/Marvin M6-S-L-CCS-696-V4.0 urdf (FUSION)/urdf/marvin_left_with_gripper.urdf (robot description, URDF)
Before this commit: robot marvin_l_with_gripper, 14 links, 13 joints
Joints:
- joint grasp_center_fixed_L: origin xyz=-0.009175 0.009190 0.202453 rpy=0 -1.5707963267948966 -0.7853981633974483 -> xyz=0 0 0.142225549599 rpy=0 -1.5707963267948966 -0.7853981633974483

File: teleop_control/vendor/tianji/Marvin M6-S-R-CCS-696-V4.0 urdf (FUSION)/urdf/marvin_right_with_gripper.urdf (robot description, URDF)
Before this commit: robot marvin_r_with_gripper, 14 links, 13 joints
Joints:
- joint grasp_center_fixed_R: origin xyz=-0.009175 0.009190 0.202453 rpy=0 -1.5707963267948966 -0.7853981633974483 -> xyz=0 0 0.142225549599 rpy=0 -1.5707963267948966 -0.7853981633974483

Commit message: tell me why？？？？？？

File: teleop_control/vendor/tianji/Marvin M6-S-L-CCS-696-V4.0 urdf (FUSION)/urdf/marvin_left_with_gripper.urdf (robot description, URDF)
Before this commit: robot marvin_l_with_gripper, 14 links, 13 joints
Joints:
- joint gripper_mount_L: origin xyz=0 0 0 rpy=0 0 2.356194490192345 -> xyz=0 0 0 rpy=0 0 -0.7853981633974483

File: teleop_control/vendor/tianji/Marvin M6-S-R-CCS-696-V4.0 urdf (FUSION)/urdf/marvin_right_with_gripper.urdf (robot description, URDF)
Before this commit: robot marvin_r_with_gripper, 14 links, 13 joints
Joints:
- joint gripper_mount_R: origin xyz=0 0 0 rpy=0 0 -0.7853981633974483 -> xyz=0 0 0 rpy=0 0 2.356194490192345

Commit message: new

File: teleop_control/vendor/tianji/Marvin M6-S-L-CCS-696-V4.0 urdf (FUSION)/urdf/marvin_left_with_gripper.urdf (robot description, URDF)
Before this commit: robot marvin_l_with_gripper, 14 links, 13 joints
Links:
- link gripper_L: geometry collision box size=0.118135551771 0.118135430406 0.108169190288; collision box size=0.203944181835 0.203945196707 0.236805177927
- link gripper_L_1: geometry collision box size=0.130341270598 0.126513042808 0.177563030733; collision mesh filename=../meshes/gripper/part_01.stl
- link gripper_L_17: geometry collision box size=0.123877538003 0.127117041309 0.177563019462; collision mesh filename=../meshes/gripper/part_17.stl
- link gripper_L_shaft: geometry collision box size=0.104995177791 0.104988304777 0.136999994218; visual mesh filename=../meshes/gripper/part_21.stl

File: teleop_control/vendor/tianji/Marvin M6-S-R-CCS-696-V4.0 urdf (FUSION)/urdf/marvin_right_with_gripper.urdf (robot description, URDF)
Before this commit: robot marvin_r_with_gripper, 14 links, 13 joints
Links:
- link gripper_R: geometry collision box size=0.118135551771 0.118135430406 0.108169190288; collision box size=0.203944181835 0.203945196707 0.236805177927
- link gripper_R_1: geometry collision box size=0.130341270598 0.126513042808 0.177563030733; collision mesh filename=../meshes/gripper/part_01.stl
- link gripper_R_17: geometry collision box size=0.123877538003 0.127117041309 0.177563019462; collision mesh filename=../meshes/gripper/part_17.stl
- link gripper_R_shaft: geometry collision box size=0.104995177791 0.104988304777 0.136999994218; visual mesh filename=../meshes/gripper/part_21.stl

Commit message: new

File: teleop_control/vendor/tianji/Marvin M6-S-L-CCS-696-V4.0 urdf (FUSION)/urdf/marvin_left_with_gripper.urdf (robot description, URDF)
Before this commit: robot marvin_l_with_gripper, 14 links, 13 joints
Links:
- link gripper_L: geometry collision mesh filename=../meshes/gripper/part_00.stl; collision mesh filename=../meshes/gripper/part_22.stl
- link gripper_L_1: geometry collision mesh filename=../meshes/gripper/part_01.stl; collision mesh filename=../meshes/gripper/part_18.stl
- link gripper_L_17: geometry collision mesh filename=../meshes/gripper/part_17.stl; collision mesh filename=../meshes/gripper/part_19.stl
- link gripper_L_shaft: geometry visual mesh filename=../meshes/gripper/part_21.stl; visual mesh filename=../meshes/gripper/part_52.stl

File: teleop_control/vendor/tianji/Marvin M6-S-R-CCS-696-V4.0 urdf (FUSION)/urdf/marvin_right_with_gripper.urdf (robot description, URDF)
Before this commit: robot marvin_r_with_gripper, 14 links, 13 joints
Links:
- link gripper_R: geometry collision mesh filename=../meshes/gripper/part_00.stl; collision mesh filename=../meshes/gripper/part_22.stl
- link gripper_R_1: geometry collision mesh filename=../meshes/gripper/part_01.stl; collision mesh filename=../meshes/gripper/part_18.stl
- link gripper_R_17: geometry collision mesh filename=../meshes/gripper/part_17.stl; collision mesh filename=../meshes/gripper/part_19.stl
- link gripper_R_shaft: geometry visual mesh filename=../meshes/gripper/part_21.stl; visual mesh filename=../meshes/gripper/part_52.stl
