Commit message: new

File: umi_collection/vendor/galaxis/galaxis_description/urdf/galaxis_hand.urdf.xacro (robot description, xacro)
@@ -28,5 +28,5 @@
   <xacro:property name="mount_z" value="0.0525"/>
   <xacro:property name="mount_roll" value="0.0"/>
-  <xacro:property name="mount_pitch" value="0.0"/>
+  <xacro:property name="mount_pitch" value="-0.7854"/>
   <xacro:property name="mount_yaw" value="0.0"/>
   <!-- JointState q is the SINGLE finger angle in radians. The full opening

Commit message: 10.28 9：57

File: umi_collection/vendor/galaxis/galaxis_description/urdf/galaxis_hand.urdf.xacro (robot description, xacro)
@@ -28,5 +28,5 @@
   <xacro:property name="mount_z" value="0.0525"/>
   <xacro:property name="mount_roll" value="0.0"/>
-  <xacro:property name="mount_pitch" value="0.0"/>
+  <xacro:property name="mount_pitch" value="-0.7854"/>
   <xacro:property name="mount_yaw" value="0.0"/>
   <!-- continuous expresses encoder-driven rotation without model limits.
